File: adaFruitKiCAD.kicad_sch (KiCad schematic)
At the start: 4 parts, among them U1 MLX90614ESF-AAA-000-TU

Commit message: Add files via upload
Parts:
- added R3, R4: R, symbol Device:R
- added U2: FSR502 FA502, Sensor_Pressure:TE_MS5837-xxBA, symbol Sensor_Pressure:MS5837-xxBA
Connections:
- net at A1.29 (GND): now also A1.9 (A0), R3.2
- net at A1.5 (+5V): now also R4.1, U2.2 (VDD)
- new net: R3.1, R4.2, U2.1 (GND)
Other:
- moved on the sheet: A1, R1, R2, U1
